File: my-corne.kicad_pcb (KiCad board)
At the start: 2 copper layers, 18 x 7 mm, 96 parts, among them SW1 SW_Push_45deg, SW10 SW_Push_45deg, SW11 SW_Push_45deg, SW12 SW_Push_45deg, SW13 SW_Push_45deg, SW14 SW_Push_45deg, SW15 SW_Push_45deg, SW16 SW_Push_45deg, SW17 SW_Push_45deg, SW18 SW_Push_45deg, SW19 SW_Push_45deg, SW2 SW_Push_45deg, SW20 SW_Push_45deg, SW21 SW_Push_45deg, SW22 SW_Push_45deg, SW23 SW_Push_45deg, SW24 SW_Push_45deg, SW25 SW_Push_45deg, SW26 SW_Push_45deg, SW27 SW_Push_45deg, SW28 SW_Push_45deg, SW29 SW_Push_45deg, SW3 SW_Push_45deg, SW30 SW_Push_45deg, SW31 SW_Push_45deg, SW32 SW_Push_45deg, SW33 SW_Push_45deg, SW34 SW_Push_45deg, SW35 SW_Push_45deg, SW36 SW_Push_45deg, SW37 SW_Push_45deg, SW38 SW_Push_45deg, SW39 SW_Push_45deg, SW4 SW_Push_45deg, SW40 SW_Push_45deg, SW41 SW_Push_45deg, SW42 SW_Push_45deg, SW43 SW_Push_45deg, SW44 SW_Push_45deg, SW45 SW_Push_45deg, SW46 RotaryEncoder_Switch, SW47 SW_Push_45deg, SW48 SW_Push_45deg, SW49 SW_Push_45deg, SW5 SW_Push_45deg, SW50 SW_Push_45deg, SW51 SW_Push_45deg, SW52 SW_Push_45deg, SW53 SW_Push_45deg, SW54 SW_Push_45deg, SW55 SW_Push_45deg, SW56 SW_Push_45deg, SW57 SW_Push_45deg, SW6 SW_Push_45deg, SW7 SW_Push_45deg, SW8 SW_Push_45deg, SW9 SW_Push_45deg, U1 RP2040_Zero

Commit message: Add files via upload
Parts:
- removed SW47, SW50: SW_Push_45deg, ScottoKeebs_MX:MX_PCB_1.50u
- removed SW48, SW52: SW_Push_45deg, ScottoKeebs_MX:MX_PCB_1.25u
- removed SW49, SW51: SW_Push_45deg, ScottoKeebs_MX:MX_PCB_ISOEnter
- removed SW53: SW_Push_45deg, ScottoKeebs_MX:MX_PCB_2.00u
- removed SW54, SW55, SW56: SW_Push_45deg, ScottoKeebs_MX:MX_PCB_1.25u_90deg
- removed SW57: SW_Push_45deg, ScottoKeebs_MX:MX_PCB_1.50u_90deg
- added D39: US2BA, ScottoKeebs_Components:Diode_SOD-123, B.Cu at (137.8, 93.8)
- added D40: US2BA, ScottoKeebs_Components:Diode_SOD-123, B.Cu at (172.0, 100.2)
- added D41: US2BA, ScottoKeebs_Components:Diode_SOD-123, B.Cu at (199.7, 96.1)
- added D42: US2BA, ScottoKeebs_Components:Diode_SOD-123, B.Cu at (221.7, 94.9)
- added D43: US2BA, ScottoKeebs_Components:Diode_SOD-123, B.Cu at (128.9, 63.1)
- added D44: US2BA, ScottoKeebs_Components:Diode_SOD-123, B.Cu at (178.3, 63.1)
- added D45: US2BA, ScottoKeebs_Components:Diode_SOD-123, B.Cu at (141.1, 82.7)
- added D46: US2BA, ScottoKeebs_Components:Diode_SOD-123, B.Cu at (166.4, 82.7)
- added J1: Conn_01x02_Socket, Connector_PinHeader_2.54mm:PinHeader_1x02_P2.54mm_Horizontal, F.Cu at (200.4, 166.6)
- added J2: Conn_01x02_Socket, Connector_PinHeader_2.54mm:PinHeader_1x02_P2.54mm_Horizontal, F.Cu at (187.9, 166.6)
- added U2: Nice_Nano_V2, ScottoKeebs_MCU:Nice_Nano_V2, F.Cu at (169.1, 44.8)
- D1, D10, D11, D12, D13, D14, D15, D16, D17, D18, D19, D2, D20, D21, D22, D23, D24, D25, D26, D27, D28, D29, D3, D30, D31, D32, D33, D34, D35, D36, D37, D38, D4, D5, D6, D7, D8, D9: value US2JA -> US2BA
- SW10, SW11: footprint ScottoKeebs_MX:MX_PCB_1.25u -> ScottoKeebs_MX:MX_PCB_1.00u
- SW21: footprint ScottoKeebs_MX:MX_PCB_1.75u -> ScottoKeebs_MX:MX_PCB_1.00u
- SW29: footprint ScottoKeebs_MX:MX_PCB_1.50u -> ScottoKeebs_MX:MX_PCB_1.00u
- SW33, SW35: footprint ScottoKeebs_MX:MX_PCB_2.75u -> ScottoKeebs_MX:MX_PCB_1.00u
- SW34: footprint ScottoKeebs_MX:MX_PCB_2.00u -> ScottoKeebs_MX:MX_PCB_1.00u
- SW39: footprint ScottoKeebs_MX:MX_PCB_1.75u -> ScottoKeebs_MX:MX_PCB_1.50u
- SW40: footprint ScottoKeebs_MX:MX_PCB_2.25u -> ScottoKeebs_MX:MX_PCB_1.50u
- SW43: value SW_Push_45deg -> RotaryEncoder_Switch; footprint ScottoKeebs_MX:MX_PCB_1.00u -> Rotary_Encoder:RotaryEncoder_Alps_EC11E-Switch_Vertical_H20mm
- SW44: value SW_Push_45deg -> RotaryEncoder_Switch; footprint ScottoKeebs_MX:MX_PCB_1.75u -> Rotary_Encoder:RotaryEncoder_Alps_EC11E-Switch_Vertical_H20mm
- SW45: value SW_Push_45deg -> SW_Reed_SPDT; footprint ScottoKeebs_MX:MX_PCB_2.25u -> Connector_PinHeader_2.54mm:PinHeader_1x03_P2.54mm_Horizontal
- SW46: value RotaryEncoder_Switch -> SW_Reed_SPDT; footprint Rotary_Encoder:RotaryEncoder_Alps_EC11E-Switch_Vertical_H20mm -> Connector_PinHeader_2.54mm:PinHeader_1x03_P2.54mm_Horizontal
- U1: value RP2040_Zero -> Nice_Nano_V2; footprint ScottoKeebs_MCU:RP2040_Zero_Flipped -> ScottoKeebs_MCU:Nice_Nano_V2; moved to F.Cu
- moved SW11 239.1 mm to (264.3, 35.7)
- moved D11 239.1 mm to (269.3, 40.2)
- moved SW12 236.3 mm to (283.4, 35.7)
- moved D12 236.3 mm to (288.4, 40.2)
- moved SW21 197.3 mm to (226.2, 47.6)
- moved D21 197.3 mm to (231.2, 52.1)
- moved SW22 189.3 mm to (245.3, 50.0)
- moved D22 189.3 mm to (250.3, 54.4)
- moved D23 188.3 mm to (269.3, 59.2)
- moved SW23 188.3 mm to (264.3, 54.8)
- moved SW24 179.0 mm to (283.4, 54.8)
- moved D24 179.0 mm to (288.4, 59.2)
- moved D32 148.0 mm to (212.2, 73.5)
- moved SW31 147.2 mm to (188.1, 71.4)
- moved D31 147.1 mm to (193.1, 75.9)
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Connections:
- D1 pad 1: R0 -> LR0
- D10 pad 1: R0 -> RR0
- D11 pad 1: R1 -> RR0
- D12 pad 1: R1 -> RR0
- D13 pad 1: R1 -> LR1
- D14 pad 1: R1 -> LR1
- D15 pad 1: R1 -> LR1
- D16 pad 1: R1 -> LR1
- D17 pad 1: R1 -> LR1
- D18 pad 1: R1 -> LR1
- D19 pad 1: R1 -> RR1
- D2 pad 1: R0 -> LR0
- D20 pad 1: R1 -> RR1
- D21 pad 1: R2 -> RR1
- D22 pad 1: R2 -> RR1
- D23 pad 1: R2 -> RR1
- D24 pad 1: R2 -> RR1
- D25 pad 1: R2 -> LR2
- D26 pad 1: R2 -> LR2
- D27 pad 1: R2 -> LR2
- D28 pad 1: R2 -> LR2
- D29 pad 1: R2 -> LR2
- D3 pad 1: R0 -> LR0
- D30 pad 1: R3 -> LR2
- D31 pad 1: R3 -> RR2
- D32 pad 1: R3 -> RR2
- D33 pad 1: R3 -> RR2
- D34 pad 1: R3 -> RR2
- D35 pad 1: R3 -> RR2
- D36 pad 1: R3 -> RR2
- D37 pad 1: R3 -> LR3
- D38 pad 1: R3 -> LR3
- D4 pad 1: R0 -> LR0
- D5 pad 1: R0 -> LR0
- D6 pad 1: R0 -> LR0
- D7 pad 1: R0 -> RR0
- D8 pad 1: R0 -> RR0
- D9 pad 1: R0 -> RR0
- SW1 pad 1: C0 -> LC0
- SW10 pad 1: C9 -> RC4
- SW11 pad 1: C0 -> RC5
- SW12 pad 1: C1 -> RC6
- SW13 pad 1: C2 -> LC0
- SW14 pad 1: C3 -> LC1
- SW15 pad 1: C4 -> LC2
- SW16 pad 1: C5 -> LC3
- SW17 pad 1: C6 -> LC4
- SW18 pad 1: C7 -> LC5
- SW19 pad 1: C8 -> RC1
- SW2 pad 1: C1 -> LC1
- SW20 pad 1: C9 -> RC2
- SW21 pad 1: C0 -> RC3
- SW22 pad 1: C1 -> RC4
- SW23 pad 1: C2 -> RC5
- SW24 pad 1: C3 -> RC6
- SW25 pad 1: C4 -> LC0
- SW26 pad 1: C5 -> LC1
- SW27 pad 1: C6 -> LC2
- SW28 pad 1: C7 -> LC3
- SW29 pad 1: C8 -> LC4
- SW3 pad 1: C2 -> LC2
- SW30 pad 1: C0 -> LC5
- SW31 pad 1: C1 -> RC1
- SW32 pad 1: C2 -> RC2
- SW33 pad 1: C3 -> RC3
- SW34 pad 1: C4 -> RC4
- SW35 pad 1: C5 -> RC5
- SW36 pad 1: C6 -> RC6
- SW37 pad 1: C7 -> LC3
- SW38 pad 1: C8 -> LC4
- SW39 pad 1: C3 -> LC5
- SW39 pad 2: Net-(D33-A) -> Net-(D39-A)
- SW4 pad 1: C3 -> LC3
- SW40 pad 1: C3 -> RC1
- SW40 pad 2: Net-(D33-A) -> Net-(D40-A)
- SW41 pad 1: C4 -> RC2
- SW41 pad 2: Net-(D34-A) -> Net-(D41-A)
- SW42 pad 1: C4 -> RC3
- SW42 pad 2: Net-(D34-A) -> Net-(D42-A)
- SW45 pad 1: C5 -> LGND
- SW45 pad 2: Net-(D35-A) -> Net-(D45-K)
- SW5 pad 1: C4 -> LC4
- SW6 pad 1: C5 -> LC5
- SW7 pad 1: C6 -> RC1
- SW8 pad 1: C7 -> RC2
- SW9 pad 1: C8 -> RC3
- U1 pad 1: R0 -> LR0
- U1 pad 10: C5 -> unconnected-(U1-7-Pad10)
- U1 pad 11: C6 -> unconnected-(U1-8-Pad11)
- U1 pad 12: C7 -> unconnected-(U1-9-Pad12)
- U1 pad 13: C8 -> unconnected-(U1-10-Pad13)
- U1 pad 14: C9 -> LC6
- U1 pad 15: unconnected-(U1-14-Pad15) -> LC5
- U1 pad 16: unconnected-(U1-15-Pad16) -> LC4
- U1 pad 17: unconnected-(U1-26-Pad17) -> LC3
- U1 pad 18: unconnected-(U1-27-Pad18) -> LC2
- U1 pad 19: C -> LC1
- U1 pad 2: R1 -> LR1
- U1 pad 20: B -> LC0
- U1 pad 22: GND -> unconnected-(U1-RST-Pad22)
- U1 pad 23: unconnected-(U1-5V-Pad23) -> LGND
- U1 pad 3: R2 -> LGND2
- U1 pad 4: R3 -> unconnected-(U1-GND-Pad4)
- U1 pad 5: C0 -> LR2
- U1 pad 6: C1 -> LR3
- U1 pad 7: C2 -> LC
- U1 pad 8: C3 -> LB
- U1 pad 9: C4 -> unconnected-(U1-6-Pad9)
Other:
- board outline removed

Commit message: Add files via upload
Parts:
- moved J1 153.0 mm to (134.3, 28.6), turned to -90 degrees
- moved J2 139.9 mm to (165.3, 28.6), turned to -90 degrees
- moved SW46 7.26 mm to (156.3, 79.9), turned to 0 degrees
- moved SW11 5.02 mm to (259.3, 35.6)
- moved SW23 5.02 mm to (259.3, 54.6)
- moved SW35 5.02 mm to (259.3, 73.7)
- moved D10 5.02 mm to (245.3, 35.3)
- moved D15 5.02 mm to (61.9, 54.3)
- moved D18 5.02 mm to (119.1, 56.7)
- moved D20 5.02 mm to (207.2, 54.3)
- moved D21 5.02 mm to (226.2, 51.9)
- moved D22 5.02 mm to (245.3, 54.3)
- moved D27 5.02 mm to (61.9, 73.4)
- moved D30 5.02 mm to (119.1, 75.7)
- moved D32 5.02 mm to (207.2, 73.4)
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Routing:
- net LC0: track 0.00 -> 170.7 mm, vias 0 -> 10
- net RR2: track 0.00 -> 165.2 mm
- net RR0: track 0.00 -> 164.8 mm
- net RR1: track 0.00 -> 152.6 mm, vias 0 -> 1
- net LC1: track 0.00 -> 150.7 mm, vias 0 -> 8
- net RC6: track 0.00 -> 147.0 mm, vias 0 -> 10
- net LR2: track 0.00 -> 140.9 mm
- net LR0: track 0.00 -> 137.4 mm
- net LC3: track 0.00 -> 137.0 mm, vias 0 -> 4
- net RR3: track 0.00 -> 136.2 mm
- net LC2: track 0.00 -> 130.0 mm, vias 0 -> 6
- net LR1: track 0.00 -> 127.8 mm, vias 0 -> 1
- net RC5: track 0.00 -> 124.9 mm, vias 0 -> 8
- net LC4: track 0.00 -> 117.1 mm, vias 0 -> 2
- net RC3: track 0.00 -> 117.0 mm, vias 0 -> 4
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Other:
- board outline added: 278.6 x 92.6 mm

Commit message: Add files via upload
Parts:
- added REF**: MountingHole_2.2mm_M2, MountingHole:MountingHole_2.2mm_M2, F.Cu at (272.1, 44.9)
- added REF**: MountingHole_2.2mm_M2, MountingHole:MountingHole_2.2mm_M2, F.Cu at (31.6, 64.0)
- added REF**: MountingHole_2.2mm_M2, MountingHole:MountingHole_2.2mm_M2, F.Cu at (195.9, 41.4)
- added REF**: MountingHole_2.2mm_M2, MountingHole:MountingHole_2.2mm_M2, F.Cu at (107.8, 80.7)
- added REF**: MountingHole_2.2mm_M2, MountingHole:MountingHole_2.2mm_M2, F.Cu at (31.6, 44.9)
- added REF**: MountingHole_2.2mm_M2, MountingHole:MountingHole_2.2mm_M2, F.Cu at (272.1, 64.0)
- added REF**: MountingHole_2.2mm_M2, MountingHole:MountingHole_2.2mm_M2, F.Cu at (107.8, 41.4)
- added REF**: MountingHole_2.2mm_M2, MountingHole:MountingHole_2.2mm_M2, F.Cu at (195.9, 80.7)
- moved D10 3.24 mm to (248.5, 35.1)
- moved D12 3.24 mm to (286.6, 39.9)
- moved D21 3.24 mm to (229.5, 51.8)
- moved D22 3.24 mm to (248.5, 54.1)
- moved D24 3.24 mm to (286.6, 58.9)
- moved D33 3.24 mm to (229.5, 70.8)
- moved D34 3.24 mm to (248.5, 73.2)
- moved D36 3.24 mm to (286.6, 78.0)
- moved D39 3.24 mm to (136.0, 93.5)
- moved D9 3.24 mm to (229.5, 32.7)
- moved SW11 3.24 mm to (262.5, 35.4)
- moved SW12 3.24 mm to (281.6, 35.4)
- moved SW21 3.24 mm to (224.4, 47.3)
- moved SW23 3.24 mm to (262.5, 54.5)
- moved SW24 3.24 mm to (281.6, 54.5)
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Routing:
- net RGND2: track 0.00 -> 42.5 mm
- net RC: track 0.00 -> 33.4 mm, vias 0 -> 2
- net RB: track 0.00 -> 31.9 mm, vias 0 -> 3
- net RR3: track 136.2 -> 130.3 mm
- net RC1: track 76.4 -> 71.1 mm
- net LC0: track 170.7 -> 175.3 mm
- net LC1: track 150.7 -> 154.6 mm
- net RC4: track 107.6 -> 106.8 mm
- net RC5: track 124.9 -> 124.0 mm
- net RC6: track 147.0 -> 146.1 mm
Other:
- outline, holes or cut-outs redrawn
