File: my-corne.kicad_sch (KiCad schematic)
At the start: 96 parts, among them J1 Conn_01x02_Socket, J2 Conn_01x02_Socket, SW1 SW_Push_45deg, SW10 SW_Push_45deg, SW11 SW_Push_45deg, SW12 SW_Push_45deg, SW13 SW_Push_45deg, SW14 SW_Push_45deg, SW15 SW_Push_45deg, SW16 SW_Push_45deg, SW17 SW_Push_45deg, SW18 SW_Push_45deg, SW19 SW_Push_45deg, SW2 SW_Push_45deg, SW20 SW_Push_45deg, SW21 SW_Push_45deg, SW22 SW_Push_45deg, SW23 SW_Push_45deg, SW24 SW_Push_45deg, SW25 SW_Push_45deg, SW26 SW_Push_45deg, SW27 SW_Push_45deg, SW28 SW_Push_45deg, SW29 SW_Push_45deg, SW3 SW_Push_45deg, SW30 SW_Push_45deg, SW31 SW_Push_45deg, SW32 SW_Push_45deg, SW33 SW_Push_45deg, SW34 SW_Push_45deg, SW35 SW_Push_45deg, SW36 SW_Push_45deg, SW37 SW_Push_45deg, SW38 SW_Push_45deg, SW39 SW_Push_45deg, SW4 SW_Push_45deg, SW40 SW_Push_45deg, SW41 SW_Push_45deg, SW42 SW_Push_45deg, SW43 RotaryEncoder_Switch, SW44 RotaryEncoder_Switch, SW45 SW_Reed_SPDT, SW46 SW_Reed_SPDT, SW5 SW_Push_45deg, SW6 SW_Push_45deg, SW7 SW_Push_45deg, SW8 SW_Push_45deg, SW9 SW_Push_45deg, U1 Nice_Nano_V2, U2 Nice_Nano_V2

Commit message: Add files via upload
Connections:
- net LR0: no longer D43.1 (K)
- net LR2: now also D43.1 (K)
- net RR0: no longer D44.1 (K)
- net RR2: now also D44.1 (K)
Other:
- note added: "1.0"
- note added: "2024/7/31"
- note added: "Diode is needed to avoid the MCU burning from an incorrectly wired battery."
- note added: "Keys & diodes matrix (left half)"
- note added: "Keys & diodes matrix (right half)"
- note added: "Left MCU"
- note added: "Left battery and switch circuit"
- note added: "Left rotary encoder"
- note added: "Right MCU"
- note added: "Right battery and switch circuit"
- note added: "Right rotary encoder"
- note added: "my-corne electrical diagram"
- moved on the sheet: D1, D10, D11, D12, D13, D14, D15, D16, D17, D18, D19, D2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

Commit message: Add files via upload
Connections:
- net LC: now also SW43.A; no longer SW43.C
- net LGND2: now also SW43.C; no longer SW43.A
- net LR0: now also D43.1 (K)
- net LR2: no longer D43.1 (K)
- net RC: now also SW44.A; no longer SW44.C
- net RGND2: now also SW44.C; no longer SW44.A
- net RR0: now also D44.1 (K)
- net RR2: no longer D44.1 (K)
