File: stroke.kicad_pcb (KiCad board)
At the start: 2 copper layers, 18 x 7 mm, 96 parts, among them SW1 SW_Push_45deg, SW10 SW_Push_45deg, SW11 SW_Push_45deg, SW12 SW_Push_45deg, SW13 SW_Push_45deg, SW14 SW_Push_45deg, SW15 SW_Push_45deg, SW16 SW_Push_45deg, SW17 SW_Push_45deg, SW18 SW_Push_45deg, SW19 SW_Push_45deg, SW2 SW_Push_45deg, SW20 SW_Push_45deg, SW21 SW_Push_45deg, SW22 SW_Push_45deg, SW23 SW_Push_45deg, SW24 SW_Push_45deg, SW25 SW_Push_45deg, SW26 SW_Push_45deg, SW27 SW_Push_45deg, SW28 SW_Push_45deg, SW29 SW_Push_45deg, SW3 SW_Push_45deg, SW30 SW_Push_45deg, SW31 SW_Push_45deg, SW32 SW_Push_45deg, SW33 SW_Push_45deg, SW34 SW_Push_45deg, SW35 SW_Push_45deg, SW36 SW_Push_45deg, SW37 SW_Push_45deg, SW38 SW_Push_45deg, SW39 SW_Push_45deg, SW4 SW_Push_45deg, SW40 SW_Push_45deg, SW41 SW_Push_45deg, SW42 SW_Push_45deg, SW43 SW_Push_45deg, SW44 SW_Push_45deg, SW45 SW_Push_45deg, SW46 RotaryEncoder_Switch, SW47 SW_Push_45deg, SW48 SW_Push_45deg, SW49 SW_Push_45deg, SW5 SW_Push_45deg, SW50 SW_Push_45deg, SW51 SW_Push_45deg, SW52 SW_Push_45deg, SW53 SW_Push_45deg, SW54 SW_Push_45deg, SW55 SW_Push_45deg, SW56 SW_Push_45deg, SW57 SW_Push_45deg, SW6 SW_Push_45deg, SW7 SW_Push_45deg, SW8 SW_Push_45deg, SW9 SW_Push_45deg, U1 RP2040_Zero

Commit message: Add files via upload
Parts:
- removed SW46: RotaryEncoder_Switch, Rotary_Encoder:RotaryEncoder_Alps_EC11E-Switch_Vertical_H20mm
- added G***: LOGO, LOGO, B.Cu at (142.9, 99.7)
- added REF**: MountingHole_2.2mm_M2, MountingHole:MountingHole_2.2mm_M2, F.Cu at (73.8, 97.3)
- added REF**: MountingHole_2.2mm_M2, MountingHole:MountingHole_2.2mm_M2, F.Cu at (219.4, 128.0)
- added REF**: MountingHole_2.2mm_M2, MountingHole:MountingHole_2.2mm_M2, F.Cu at (69.1, 140.2)
- added REF**: MountingHole_2.2mm_M2, MountingHole:MountingHole_2.2mm_M2, F.Cu at (231.0, 102.1)
- moved D10 159.5 mm to (245.6, 94.5)
- moved D9 132.9 mm to (219.4, 89.9)
- moved D8 109.4 mm to (200.6, 79.5)
- moved D7 97.0 mm to (171.7, 89.9)
- moved D6 87.9 mm to (152.7, 89.9)
- moved D5 85.9 mm to (129.5, 92.0)
- moved D4 85.8 mm to (114.6, 89.9)
- moved D3 81.1 mm to (95.0, 75.9)
- moved D21 60.0 mm to (55.0, 137.2)
- moved D22 60.0 mm to (81.2, 132.4)
- moved D23 60.0 mm to (100.3, 125.3)
- moved D24 60.0 mm to (128.8, 127.7)
- moved D25 60.0 mm to (147.9, 127.7)
- moved D26 60.0 mm to (166.9, 127.7)
- moved D27 60.0 mm to (186.0, 127.7)
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Routing:
- net R3: track 0.00 -> 283.7 mm, vias 0 -> 3
- net R2: track 0.00 -> 249.8 mm, vias 0 -> 1
- net R1: track 0.00 -> 248.7 mm, vias 0 -> 1
- net R0: track 0.00 -> 243.5 mm
- net C7: track 0.00 -> 171.0 mm, vias 0 -> 3
- net C8: track 0.00 -> 166.9 mm, vias 0 -> 3
- net C0: track 0.00 -> 163.8 mm, vias 0 -> 7
- net C1: track 0.00 -> 156.9 mm, vias 0 -> 5
- net C9: track 0.00 -> 152.3 mm, vias 0 -> 5
- net C2: track 0.00 -> 144.4 mm, vias 0 -> 3
- net C6: track 0.00 -> 123.7 mm, vias 0 -> 3
- net C3: track 0.00 -> 105.8 mm, vias 0 -> 1
- net C5: track 0.00 -> 94.5 mm, vias 0 -> 1
- net C4: track 0.00 -> 75.3 mm
- net Net-(D34-A): track 0.00 -> 34.5 mm
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- added copper zone on B.Cu, net (none)
- added copper zone on F.Cu, net (none)
Other:
- board size 18 x 7 mm -> 219.1 x 90.5 mm
